File: main/battery_temp_sensors.kicad_sch (KiCad schematic)
At the start: 3 parts, among them U3 ESP32-DevKitC

Commit message: added logos, oranised sheets, final version
Other:
- company: (none) -> Designers: Krzysztof Grajek, Wojtek Kołodziej
- moved on the sheet: A3, D36V6F25, U3
